File: hardware/ESC.kicad_sch (KiCad schematic)
At the start: 36 parts, among them Q1 DOY180N03T, Q2 DOY180N03T, Q3 DOY180N03T, Q4 DOY180N03T, Q5 DOY180N03T, Q6 DOY180N03T, U2 AT32F421G8U7, U3 NSG2065Q

Commit message: schematics: fill Manufacturer on every part, drop empty LCSC_Part stub
Every placed part with an LCSC number now carries LCSC + Manufacturer + MPN,
manufacturer names taken from the LCSC catalogue (18 parts backfilled; the
catalogue MPN matched the existing MPN field on all of them). Feeds the new
fab-agnostic BOM export in OpenDrone-Scripts for quoting outside JLCPCB.

kicad-skip reflowed both files on write, so the text diff is large; an
S-expression structural diff against the originals shows the only content
change is the property add/remove, and ERC is identical before and after
(334 violations, same categories).

Co-Authored-By: Claude Fable 5 <noreply@anthropic.com>
Parts:
- C32, C36, C53: Manufacturer (none) -> Samsung Electro-Mechanics
- C48, C49, C50, C57: Manufacturer (none) -> muRata
- Q1, Q2, Q3, Q4, Q5, Q6: Manufacturer (none) -> DOINGTER
- R16, R17, R21, R22, R23, R24, R26, R29, R32: Manufacturer (none) -> UNI-ROYAL
- R18, R19, R20, R25, R27, R28, R30, R31, R33, R74: Manufacturer (none) -> YAGEO
- U3: Manufacturer (none) -> WXNSIC
