File: hardware/4in1-mini.kicad_sch (KiCad schematic)
At the start: 26 parts, among them J1 SM08B-SRSS-TB, U1 TLV76733DRVR, U12 INA186A3IDCKR, U13 LMR54406DBVR, U5 FTC160808S4R7MBCA

Commit message: schematics: fill Manufacturer on every part, drop empty LCSC_Part stub
Every placed part with an LCSC number now carries LCSC + Manufacturer + MPN,
manufacturer names taken from the LCSC catalogue (18 parts backfilled; the
catalogue MPN matched the existing MPN field on all of them). Feeds the new
fab-agnostic BOM export in OpenDrone-Scripts for quoting outside JLCPCB.

kicad-skip reflowed both files on write, so the text diff is large; an
S-expression structural diff against the originals shows the only content
change is the property add/remove, and ERC is identical before and after
(334 violations, same categories).

Co-Authored-By: Claude Fable 5 <noreply@anthropic.com>
Parts:
- C1, C42, C43, C52, C54, C86, CL32: Manufacturer (none) -> Samsung Electro-Mechanics
- C51, R118: Manufacturer (none) -> YAGEO
- C69, C70, C71, C72, C93, C94: Manufacturer (none) -> muRata
- J1: Manufacturer (none) -> JST
- R119: Manufacturer (none) -> RALEC
- R73, R91, R92: Manufacturer (none) -> UNI-ROYAL
- Rsense2: Manufacturer (none) -> Yezhan
- U13: LCSC Part C5219316 -> (none)
- U5: Manufacturer (none) -> cjiang

Commit message: Swap bulk caps to FH 1206B475K500NT 4.7uF 50V (C29823)
Replaces Samsung CL31B106KBHNNNE 10uF (C89632) on schematic symbol
CL32. Board file 4in1-mini.kicad_pcb also swapped (22 footprints) but
left uncommitted: it carries unrelated WIP via/routing changes.

Co-Authored-By: Claude Fable 5 <noreply@anthropic.com>
Parts:
- CL32: value 10uF -> 4.7uF; Cost 0.05129 -> (none); LCSC C89632 -> C29823; MPN CL31B106KBHNNNE -> 1206B475K500NT; Manufacturer Samsung Electro-Mechanics -> FH

Commit message: Swap bulk caps to CCTC TCC1206X7R475K500HT (C380366)
FH C29823 was picked for its JLC-basic price; at LCSC retail it costs
USD 0.19/pc and we are no longer using JLCPCB assembly. CCTC part is
~USD 0.073/pc at 4k+ volume, same 4.7uF 10% 50V X7R 1206 class.
Fields only (LCSC/MPN/Manufacturer), no value, footprint or net changes.

Co-Authored-By: Claude Fable 5 <noreply@anthropic.com>
Parts:
- CL32: LCSC C29823 -> C380366; MPN 1206B475K500NT -> TCC1206X7R475K500HT; Manufacturer FH -> CCTC
